File: PCB/Aurora/Aurora.kicad_sch (KiCad schematic)
At the start: 0 parts

Commit message: Schema + PCB
Parts:
- added AL1: ~, SamacSys:PSK-10E-5, symbol SamacSys:PSK-10E-5
- added C1, C2, C4: GXT21BR71A475KE13L, CAPC2012X140N, symbol SamacSys:GXT21BR71A475KE13L
- added C3, C5: 100nF, Capacitor_SMD:C_0402_1005Metric, symbol SamacSys_Parts:AC0402KRX7R7BB104
- added C6, C7, C8: CGA4J1X7R0J106K125AC, CGA4J2NP01H223J125AA, symbol SamacSys:CGA4J1X7R0J106K125AC
- added D1, D2, D3: SS14, DIOM5227X270N, symbol SamacSys:SS14
- added F1: 3403.0166.24, SamacSys:3403016624, symbol SamacSys:3403.0166.24
- added IC1: TPS73533DRVT, SON65P200X200X80-7N, symbol SamacSys:TPS73533DRVT
- added IC2: USBLC6-2SC6, SamacSys:SOT95P280X145-6N, symbol SamacSys:USBLC6-2SC6
- added IC3: STM32G0B1KBU6, Package_DFN_QFN:QFN-32-1EP_5x5mm_P0.5mm_EP3.45x3.45mm, symbol SamacSys:STM32G0B1KBU6
- added IC4, IC5, IC6: AL8860WT-7, SOT95P280X100-5N, symbol SamacSys:AL8860WT-7
- added J1: 1190297, 1190297, symbol SamacSys:1190297
- added J2: USB4940-00-A, USB494000A, symbol SamacSys:USB4940-00-A
- added J3: FTSH-107-01-F-DV-K, FTSH-107-XX-YYY-DV-K, symbol SamacSys:FTSH-107-01-F-DV-K
- added J4: 1190297, SamacSys:Pad_Connector_2, symbol SamacSys:Pad_Connector_2
- added J5: 1751183, 1751183, symbol SamacSys:1751183
- added L1, L2, L3: PA4332.472NLT, PA4332472NLT, symbol SamacSys:PA4332.472NLT
- added LED1, LED2: ~, SamacSys:OT-3RGB-C30, symbol SamacSys:OT-3RGB-C30
- added Q1, Q10, Q2, Q3, Q4, Q5, Q6, Q7, Q8, Q9: ~, SamacSys:TLP2303TPLE, symbol SamacSys:TLP2303TPLE
- added R1, R14, R15, R16, R17, R18, R2, R3, R4, R5: 5.1R, RESC5025X120N, symbol SamacSys:35025K1FT
- added R10, R11, R12, R13, R20, R21, R22, R23, R24, R9: 3.3R, SamacSys:RESC1608X55N, symbol SamacSys:CR0603-FX-3301ELF
- added R19, R7: CR0603-FX-5101ELF, RESC1608X55N, symbol SamacSys:CR0603-FX-5101ELF
- added R25, R26, R27: 100R, Resistor_SMD:R_0603_1608Metric, symbol SamacSys:SFR03EZPJ101
- added R28, R29, R30: 0.16R, Resistor_SMD:R_0603_1608Metric, symbol SamacSys:RL0603FR-070R16L
- added R6: MCT0603MC3302FP500, RESC1608X55N, symbol SamacSys:MCT0603MC3302FP500
- added R8: ERJ-P08F8202V, SamacSys:ERJP08__1206_, symbol SamacSys:ERJ-P08F8202V
- added S1: SPST, SamacSys:TS09-63-25-WT-160-SMT-TR, symbol SamacSys:TS09-63-25-WT-160-SMT-TR
Connections:
- net 3.3V: now also C2.1, C4.1, C5.1, IC1.1 (OUT), IC3.4 (VDD/VDDA), J3.3, Q1.6 (Vcc), Q10.6 (Vcc), Q2.6 (Vcc), Q3.6 (Vcc), Q4.6 (Vcc), Q5.6 (Vcc), Q6.6 (Vcc), Q7.6 (Vcc), Q8.6 (Vcc), Q9.6 (Vcc), R10.2, R11.2, R12.2, R13.2, R20.2, R21.2, R22.2, R23.2, R24.2, R9.2
- new net: Q10.1 (Anode), R18.2
- new net: Q1.1 (Anode), R1.2
- new net: IC2.1 (I/O1_1), J2.A7 (DN1), J2.B7 (DN2)
- new net: IC2.3 (I/O2_1), J2.A6 (DP1), J2.B6 (DP2)
- new net: IC2.5 (VBUS), J2.A4 (VBUS_1), J2.B4 (VBUS_2), R6.1
- new net: D2.2, IC5.1 (SW), L2.2
- new net: F1.1, J1.1, J1.3
- new net: AL1.2 (N), J1.2, J1.4
- new net: J2.A5 (CC1), R7.2
- new net: J2.B5 (CC2), R19.1
- new net: D1.2, IC4.1 (SW), L1.2
- new net: Q9.1 (Anode), R17.2
- new net: Q5.1 (Anode), R5.2
- new net: AL1.1 (L), F1.2
- new net: D3.2, IC6.1 (SW), L3.2
- new net: Q6.1 (Anode), R14.2
- new net: Q8.1 (Anode), R16.2
- new net: Q3.1 (Anode), R3.2
- new net: IC3.21 (PA10), R25.1
- new net: Q7.1 (Anode), R15.2
- new net: Q2.1 (Anode), R2.2
- new net: IC3.18 (PA8), R27.1
- new net: IC3.19 (PA9), R26.1
- new net: Q4.1 (Anode), R4.2
- new net 5V: AL1.4 ((+)), C1.2, C3.2, C6.1, C7.1, C8.1, D1.1, D2.1, D3.1, IC1.4 (EN), IC1.6 (IN), IC4.5 (VIN), IC5.5 (VIN), IC6.5 (VIN), J4.1, R28.2, R29.2, R30.2
- new net CH_BLUE: IC5.3 (CTRL), R25.2
- new net CH_GREEN: IC4.3 (CTRL), R26.2
- new net CH_RED: IC6.3 (CTRL), R27.2
- new net GND: AL1.3 ((-)), C1.1, C2.2, C3.1, C4.2, C5.2, C6.2, C7.2, C8.2, IC1.3 (GND), IC1.7 (EP), IC3.33 (EP), IC3.5 (VSS/VSSA), IC4.2 (GND), IC5.2 (GND), IC6.2 (GND), J2.A1 (GND_1), J2.B1 (GND_2), J2.S1 (GND_3), J2.S2 (GND_4), J2.S3 (GND_5), J2.S4 (GND_6), J3.11, J3.2, J3.5, J3.7, J4.2, Q1.4 (GND), Q10.4 (GND), Q2.4 (GND), Q3.4 (GND), Q4.4 (GND), Q5.4 (GND), Q6.4 (GND), Q7.4 (GND), Q8.4 (GND), Q9.4 (GND), R19.2, R7.1, R8.2, S1.1
- new net I_{0}: J5.11, R1.1
- new net I_{1}: J5.10, R2.1
- new net I_{2}: J5.9, R3.1
- new net I_{3}: J5.8, R4.1
- new net I_{4}: J5.7, R5.1
- new net I_{5}: J5.6, R14.1
- new net I_{6}: J5.5, R15.1
- new net I_{7}: J5.4, R16.1
- new net I_{8}: J5.3, R17.1
- new net I_{9}: J5.2, R18.1
- new net I_{COMMON}: J5.1, Q1.3 (Cathode), Q10.3 (Cathode), Q2.3 (Cathode), Q3.3 (Cathode), Q4.3 (Cathode), Q5.3 (Cathode), Q6.3 (Cathode), Q7.3 (Cathode), Q8.3 (Cathode), Q9.3 (Cathode)
- new net In_{0}: IC3.7 (PA0), Q1.5 (Output), R9.1
- new net In_{1}: IC3.8 (PA1), Q2.5 (Output), R10.1
- new net In_{2}: IC3.9 (PA2), Q3.5 (Output), R11.1
- new net In_{3}: IC3.10 (PA3), Q4.5 (Output), R12.1
- new net In_{4}: IC3.11 (PA4), Q5.5 (Output), R13.1
- new net In_{5}: IC3.12 (PA5), Q6.5 (Output), R20.1
- new net In_{6}: IC3.13 (PA6), Q7.5 (Output), R21.1
- new net In_{7}: IC3.14 (PA7), Q8.5 (Output), R22.1
- new net In_{8}: IC3.15 (PB0), Q9.5 (Output), R23.1
- new net In_{9}: IC3.16 (PB1), Q10.5 (Output), R24.1
- new net LED(B)+: L2.1, LED1.6, LED2.6
- new net LED(B)-: IC5.4 (SET), LED1.5, LED2.5, R29.1
- new net LED(G)+: L1.1, LED1.4, LED2.4
- new net LED(G)-: IC4.4 (SET), LED1.3, LED2.3, R28.1
- new net LED(R)+: L3.1, LED1.2, LED2.2
- new net LED(R)-: IC6.4 (SET), LED1.1, LED2.1, R30.1
- new net NRST: IC3.6 (PF2-NRST), J3.12, S1.2
- new net SYS_SWCLK: IC3.25 (PA14-BOOT0), J3.6
- new net SYS_SWDIO: IC3.24 (PA13), J3.4
- new net USB_DN: IC2.6 (I/O1_2), IC3.22 (PA11[PA9])
- new net USB_DP: IC2.4 (I/O2_2), IC3.23 (PA12[PA10])
- new net USB_VBUS_Sense: IC3.20 (PC6), R6.2, R8.1
- no-connect marks 0 -> 11
Other:
- removed sheet Alimentation
- removed sheet MCU
- note added: "Ventilateur"
