File: PCB/Aurora/alimentation.kicad_sch (KiCad schematic)
At the start: 19 parts, among them IC1 DCP3603BCMR, J1 1190297, Q1 FQD8P10TM-F085

Commit message: Schema + PCB
Parts:
- removed C1: C1608X7R1H104K080AA, SamacSys_Parts:CAPC1608X80N, symbol SamacSys_Parts:C1608X7R1H104K080AA
- removed C2, C3: C2012X5R1E226M125AC, CAPC2012X145N, symbol SamacSys_Parts:C2012X5R1E226M125AC
- removed C4: C2012X7R1H225K125AC, CAPC2012X145N, symbol SamacSys_Parts:C2012X7R1H225K125AC
- removed C5: APZ0609470M050R, CAPAE660X980N, symbol SamacSys_Parts:APZ0609470M050R
- removed C6: GCM21BM8EH475KE08L, CAPC2012X145N, symbol SamacSys_Parts:GCM21BM8EH475KE08L
- removed D1: SZ1SMA5929BT3G, DIOM5226X220N, symbol SamacSys_Parts:SZ1SMA5929BT3G
- removed D2: PESD1IVN27-UX, PESD1IVN27UX, symbol SamacSys_Parts:PESD1IVN27-UX
- removed F1: SF-0603SP100-2, FUSC1608X55N, symbol SamacSys_Parts:SF-0603SP100-2
- removed IC1: DCP3603BCMR, SOT95P280X125-6N, symbol SamacSys_Parts:DCP3603BCMR
- removed L1: XAL6060-562MEC, XAL6060562MEC, symbol SamacSys_Parts:XAL6060-562MEC
- removed L2: LQM21DH100M70L, LQM21DN220N00L, symbol SamacSys_Parts:LQM21DH100M70L
- removed Q1: FQD8P10TM-F085, FQD20N06TM, symbol SamacSys_Parts:FQD8P10TM-F085
- removed R1: CRCW120630K0FKEAC, RESC3216X60N, symbol SamacSys_Parts:CRCW120630K0FKEAC
- removed R2: CRCW080586K6FKEA, RESC2012X50N, symbol SamacSys_Parts:CRCW080586K6FKEA
- removed R3, R4: 10kR, SamacSys_Parts:RESC3225X60N, symbol SamacSys_Parts:CRCW121010K0JNEAIF
- removed R5: CR1206-FX-1473ELF, RESC3216X75N, symbol SamacSys_Parts:CR1206-FX-1473ELF
- added AL1: ~, SamacSys:PSK-10E-5, symbol SamacSys:PSK-10E-5
- added C1, C3: 4.7uF, SamacSys_Parts:C0402C104J4RACTU, symbol SamacSys_Parts:C0402C475K8PACTU
- added C2: 100nF, Capacitor_SMD:C_0402_1005Metric, symbol SamacSys_Parts:AC0402KRX7R7BB104
- added F?: 3403.0166.24, SamacSys:3403016624, symbol SamacSys:3403.0166.24
- added IC3: TPS73533DRVT, SON65P200X200X80-7N, symbol SamacSys:TPS73533DRVT
Connections:
- net 3.3V: now also C1.1, IC3.1 (OUT)
- net GND: now also AL1.3 ((-)), C1.2, C2.1, C3.1, IC3.3 (GND), IC3.7 (EP); no longer J1.2, J1.4
- net at J1.1, J1.3: now also F?.1
- new net: AL1.1 (L), F?.2
- new net: AL1.2 (N), J1.2, J1.4
- new net 5V: AL1.4 ((+)), C2.2, C3.2, IC3.4 (EN), IC3.6 (IN)
- no-connect marks 0 -> 1
